File: ASD2003.brd (EAGLE design)
At the start: 22.5 x 22.5 mm, 23 parts, among them J1 PIN_1X.1"1, J10 PIN_1X.1"1, J11 PIN_1X.1"1, J12 DF12-32-DS, J13 PIN_1X.1"1, J14 PIN_1X.1"1, J15 PIN_1X.1"1, J16 PIN_1X.1"1, J17 PIN_1X.1"1, J18 PIN_1X.1"1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

Commit message: Updated to Rev 3
Routing:
- net GND: track 0.50 -> 2.79 mm, vias 0 -> 1
- net VCC: track 26.4 -> 25.6 mm
- net VBATT: vias 0 -> 2
Other:
- board text added: "0"
- board text added: "2"
- board text added: "3"
- board text added: "4"
- board text added: "A0"
- board text added: "A1"
- board text added: "A2"
- board text added: "A3"
- board text added: "A4"
- board text added: "A5"
- board text added: "REV 3"
- board text removed: "AD0"
- board text removed: "AD1"
- board text removed: "AD2"
- board text removed: "AD3"
- board text removed: "IO0"
- board text removed: "IO1"
- board text removed: "IO2"
- board text removed: "IO3"
- board text removed: "IO4"
- board text removed: "REV 1"
- board text removed: "SCL"
- board text removed: "SDA"
